File: pixhawk_shield/pixhawk_shield.sch (KiCad schematic (older format))
At the start: 11 parts

Commit message: no message
Parts:
- added J1: Conn_D8R_G, Pin_Headers:Pin_Header_Straight_1x08_Pitch2.54mm, symbol Connector_Generic:Conn_01x08
- added J10, J13: MAIN_OUT_3, Connectors_Molex:Molex_SPOX-5267_22-03-5035_03x2.54mm_Straight, symbol Connector_Generic:Conn_01x03
- added J11, J14: MAIN_OUT_5, Connectors_Molex:Molex_SPOX-5267_22-03-5035_03x2.54mm_Straight, symbol Connector_Generic:Conn_01x03
- added J12, J15: MAIN_OUT_7, Connectors_Molex:Molex_SPOX-5267_22-03-5035_03x2.54mm_Straight, symbol Connector_Generic:Conn_01x03
- added J16: MAIN_OUT_2, Connectors_Molex:Molex_SPOX-5267_22-03-5035_03x2.54mm_Straight, symbol Connector_Generic:Conn_01x03
- added J17, J20: MAIN_OUT_4, Connectors_Molex:Molex_SPOX-5267_22-03-5035_03x2.54mm_Straight, symbol Connector_Generic:Conn_01x03
- added J18, J21: MAIN_OUT_6, Connectors_Molex:Molex_SPOX-5267_22-03-5035_03x2.54mm_Straight, symbol Connector_Generic:Conn_01x03
- added J19, J22: MAIN_OUT_8, Connectors_Molex:Molex_SPOX-5267_22-03-5035_03x2.54mm_Straight, symbol Connector_Generic:Conn_01x03
- added J2: Conn_D8R_V, Pin_Headers:Pin_Header_Straight_1x08_Pitch2.54mm, symbol Connector_Generic:Conn_01x08
- added J3: Conn_D8R_S, Pin_Headers:Pin_Header_Straight_1x08_Pitch2.54mm, symbol Connector_Generic:Conn_01x08
- added J4: Conn_PPM_IN, Pin_Headers:Pin_Header_Straight_1x10_Pitch2.54mm, symbol Connector_Generic:Conn_01x10
- added J8: MAIN_OUT_1, Connectors_Molex:Molex_SPOX-5267_22-03-5035_03x2.54mm_Straight, symbol Connector_Generic:Conn_01x03
- added J9: POWER, Connector_Hirose:Hirose_DF13-06P-1.25DSA_1x06_P1.25mm_Vertical, symbol Connector_Generic:Conn_01x06
- J5: renamed from J?; value Conn_01x03 -> Conn_PPM_OUT
- J6: renamed from J?; value Conn_01x18 -> Pixhawk
- gave numbers to parts that had none: 9
Connections:
- net +5V: now also J5.2 (Pin_2), J10.2 (Pin_2), J11.2 (Pin_2), J12.2 (Pin_2), J13.2 (Pin_2), J14.2 (Pin_2), J15.2 (Pin_2), J16.2 (Pin_2), J17.2 (Pin_2), J18.2 (Pin_2), J19.2 (Pin_2), J2.1 (Pin_1), J2.2 (Pin_2), J2.3 (Pin_3), J2.4 (Pin_4), J2.5 (Pin_5), J2.6 (Pin_6), J2.7 (Pin_7), J2.8 (Pin_8), J20.2 (Pin_2), J21.2 (Pin_2), J22.2 (Pin_2), J4.2 (Pin_2), J8.2 (Pin_2)
- net GND: now also J5.1 (Pin_1), J1.1 (Pin_1), J1.2 (Pin_2), J1.3 (Pin_3), J1.4 (Pin_4), J1.5 (Pin_5), J1.6 (Pin_6), J1.7 (Pin_7), J1.8 (Pin_8), J10.1 (Pin_1), J11.1 (Pin_1), J12.1 (Pin_1), J13.1 (Pin_1), J14.1 (Pin_1), J15.1 (Pin_1), J16.1 (Pin_1), J17.1 (Pin_1), J18.1 (Pin_1), J19.1 (Pin_1), J20.1 (Pin_1), J21.1 (Pin_1), J22.1 (Pin_1), J4.1 (Pin_1), J8.1 (Pin_1)
- net SBUS: now reaches J5.3 (Pin_3)
- net SBUS: now also J6.16 (Pin_16)
- net MAIN_OUT_3: now reaches J6.10 (Pin_10)
- net MAIN_OUT_3: now also J10.3 (Pin_3)
- net MAIN_OUT_4: now reaches J6.11 (Pin_11)
- net MAIN_OUT_4: now also J17.3 (Pin_3)
- net MAIN_OUT_5: now reaches J6.12 (Pin_12)
- net MAIN_OUT_5: now also J11.3 (Pin_3)
- net MAIN_OUT_6: now reaches J6.13 (Pin_13)
- net MAIN_OUT_6: now also J18.3 (Pin_3)
- net MAIN_OUT_7: now reaches J6.14 (Pin_14)
- net MAIN_OUT_7: now also J12.3 (Pin_3)
- net MAIN_OUT_8: now reaches J6.15 (Pin_15)
- net MAIN_OUT_8: now also J19.3 (Pin_3)
- net AUX_OUT_1: now reaches J6.2 (Pin_2)
- net AUX_OUT_1: now also J13.3 (Pin_3)
- net AUX_OUT_2: now reaches J6.3 (Pin_3)
- net AUX_OUT_2: now also J20.3 (Pin_3)
- net AUX_OUT_3: now reaches J6.4 (Pin_4)
- net AUX_OUT_3: now also J14.3 (Pin_3)
- net AUX_OUT_4: now reaches J6.5 (Pin_5)
- net AUX_OUT_4: now also J21.3 (Pin_3)
- net AUX_OUT_5: now reaches J6.6 (Pin_6)
- net AUX_OUT_5: now also J15.3 (Pin_3)
- net AUX_OUT_6: now reaches J6.7 (Pin_7)
- net AUX_OUT_6: now also J22.3 (Pin_3)
- net MAIN_OUT_1: now reaches J6.8 (Pin_8)
- net MAIN_OUT_1: now also J8.3 (Pin_3)
- net MAIN_OUT_2: now reaches J6.9 (Pin_9)
- net MAIN_OUT_2: now also J16.3 (Pin_3)
- new net: J3.8 (Pin_8), J4.10 (Pin_10)
- new net: J3.1 (Pin_1), J4.3 (Pin_3)
- new net: J3.2 (Pin_2), J4.4 (Pin_4)
- new net: J3.3 (Pin_3), J4.5 (Pin_5)
- new net: J3.4 (Pin_4), J4.6 (Pin_6)
- new net: J3.5 (Pin_5), J4.7 (Pin_7)
- new net: J3.6 (Pin_6), J4.8 (Pin_8)
- new net: J3.7 (Pin_7), J4.9 (Pin_9)
Other:
- moved on the sheet: J5, J6
